Commit message: added fixed urdf

File: share/urdf/pepper.urdf (robot description, URDF)
Before this commit: robot JulietteY20MP, 84 links, 83 joints
Links:
- removed link ImuBaseGyrometer_frame
Joints:
- removed joint GyrometerBase_sensor_fixedjoint
- joint AccelerometerBase_sensor_fixedjoint: origin xyz=0 0 -0.3 rpy=0 0 0 -> xyz=0.0147 -0.0017 -0.26319 rpy=0 0 0
- joint CameraBottom_sensor_fixedjoint: origin xyz=0.0936 0 0.0616 rpy=0 0.698132 0 -> xyz=0.09262 0 0.06177 rpy=0 0.698132 0
- joint CameraTop_sensor_fixedjoint: origin xyz=0.0868 0 0.1631 rpy=0 0 0 -> xyz=0.08601 0 0.16284 rpy=0 0 0
- joint LaserSensor/Front_sensor_fixedjoint: origin xyz=0.0562 0 -0.0692 rpy=0 0.349044 0 -> xyz=0.0562 0 -0.0692 rpy=0 0.349066 0
- joint LaserSensor/Left_sensor_fixedjoint: origin xyz=-0.018 0.0899 -0.0759 rpy=8.34035e-09 0.191982 1.5708 -> xyz=-0.018 0.0899 -0.0759 rpy=0 0.349066 1.5708
- joint LaserSensor/Right_sensor_fixedjoint: origin xyz=-0.018 -0.0899 -0.0759 rpy=4.08851e-07 0.191857 -1.60746 -> xyz=-0.018 -0.0899 -0.0759 rpy=0 0.349066 -1.5708
- joint LaserSensor/Shovel_sensor_fixedjoint: origin xyz=0.0562 0 -0.0692 rpy=0 0.349044 0 -> xyz=0.0562 0 -0.0692 rpy=0 0.349066 0
- joint LaserSensor/VerticalLeft_sensor_fixedjoint: origin xyz=0.0562 0 -0.0692 rpy=0 0.349044 0 -> xyz=0.0562 0 -0.0692 rpy=0 0.349066 0
- joint LaserSensor/VerticalRight_sensor_fixedjoint: origin xyz=0.0562 0 -0.0692 rpy=0 0.349044 0 -> xyz=0.0562 0 -0.0692 rpy=0 0.349066 0

Commit message: fixed urdf

File: share/urdf/pepper.urdf (robot description, URDF)
Before this commit: robot JulietteY20MP, 83 links, 82 joints
Links:
- removed link base_link
- added link Lgrasp_frame
- added link l_grasp_frame, mass 0
- added link r_grasp_frame, mass 0
- added link torso_base
Joints:
- removed joint base_link_fixedjoint
- added joint LGrasp: type fixed, parent l_wrist, child l_grasp_frame, origin xyz=0.05 0 0 rpy=-3.1415 0 1.5707, axis 1.0 0 0, limit lower=0.02 upper=0.98 effort=0.144 velocity=12.56
- added joint Lgrasp_frame_joint: type fixed, parent l_wrist, child Lgrasp_frame, origin xyz=0.070 0 0 rpy=3.1415 0 1.5707
- added joint RGrasp: type fixed, parent r_wrist, child r_grasp_frame, origin xyz=0.05 0 0 rpy=-3.1415 0 1.5707, axis 1.0 0 0, limit lower=0.02 upper=0.98 effort=0.144 velocity=12.56
- added joint torso_base_fixedjoint: type fixed, parent torso_base, child torso, origin xyz=-2e-05 0 0.139 rpy=0 0 0, axis 0 0 0
- joint HipPitch: child Pelvis -> Hip; origin xyz=0 0 -0.079 rpy=0 0 0 -> xyz=0 0 0.268 rpy=0 0 0; parent Hip -> Pelvis
- joint HipRoll: child Hip -> torso_base; origin xyz=2e-05 0 -0.139 rpy=0 0 0 -> xyz=0 0 0.079 rpy=0 0 0; parent torso -> Hip
- joint KneePitch: child Tibia -> Pelvis; origin xyz=0 0 -0.268 rpy=0 0 0 -> xyz=0 0 0 rpy=0 0 0; parent Pelvis -> Tibia
- joint base_footprint_joint: child base_footprint -> Tibia; origin xyz=0 0 -0.334 rpy=0 0 0 -> xyz=0 0 0.334 rpy=0 0 0; parent Tibia -> base_footprint
